File: schematics/music_gadget_encoder.kicad_pcb (KiCad board)
At the start: 2 copper layers, 96.5 x 49.9 mm, 249 parts, among them IC1 TLC5926IPWPR, J6 Conn_01x02_Male, Q1 DMG9933USD-13, Q2 DMG9933USD-13, Q3 DMG9933USD-13, Q4 DMG9933USD-13, Q5 DMG9933USD-13, SW1 SW_Push, SW2 SW_Push, SW3 SW_Push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

Commit message: update pcb
Connections:
- J_LEFT1 pad 3: /USART4_RX -> /USART4_TX
- J_LEFT1 pad 4: /USART4_TX -> /USART4_RX
- J_TOP1 pad 3: /USART3_RX -> /USART3_TX
- J_TOP1 pad 4: /USART3_TX -> /USART3_RX
Routing:
- net /USART3_TX: track 20.1 -> 25.4 mm
- net /USART4_TX: track 32.3 -> 35.5 mm
- net /USART3_RX: track 16.1 -> 19.0 mm
- net /USART4_RX: track 35.4 -> 33.3 mm
- net VCC: track 500.7 -> 499.0 mm
- net GND: vias 246 -> 244
